File: spi-onboard-prog/spi-onboard-prog.kicad_sch (KiCad schematic)
At the start: 29 parts, among them CN1 USERPORT-C64-CONN, IC1 74LS07, IC4 74164DLS, P2 PETUSERPORT

Commit message: layout work on onboard spi prog
Connections:
- net GND: now also IC1.7 (GND), IC4.7 (GND)
- net VCC: now also IC1.14 (VCC), IC4.14 (VCC)

Commit message: move spi onboard prog to draft spi userport
Parts:
- added unit 7 of IC1
- added unit 2 of IC4
Connections:
- net GND: now also IC1.7 (GND), IC4.7 (GND); no longer IC1.7 (GND), IC4.7 (GND)
- net VCC: now also IC1.14 (VCC), IC4.14 (VCC); no longer IC1.14 (VCC), IC4.14 (VCC)

Commit message: onboard flash prog
Parts:
- C11: LCSC (none) -> C14663
- C3: LCSC (none) -> C96123
Changed lines of the file:
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@@
+			)
+		)
+		(property "LCSC" "C96123"
+			(at 139.065 201.0409 0)
+			(effects
+				(font
+					(size 1.27 1.27)
+				)
+				(hide yes)
 			)
 		)
@@
 			)
 		)
+		(property "LCSC" "C14663"
+			(at 125.984 201.549 0)
+			(effects
+				(font
+					(size 1.27 1.27)
+				)
+				(hide yes)
+			)
+		)
